Commit message: fix for panda mimic

File: src/curobo/content/assets/robot/franka_description/franka_panda.urdf (robot description, URDF)
Before this commit: robot panda, 14 links, 13 joints
Joints:
- joint panda_finger_joint2: mimic joint=panda_finger_joint1 -> (none)

File: src/curobo/content/assets/robot/franka_description/franka_panda_mobile_xy_tz.urdf (robot description, URDF)
Before this commit: robot panda, 19 links, 18 joints
Joints:
- joint panda_finger_joint2: mimic joint=panda_finger_joint1 -> (none)

File: src/curobo/content/assets/robot/franka_description/franka_test.urdf (robot description, URDF)
Before this commit: robot panda, 14 links, 13 joints
Joints:
- joint panda_finger_joint2: mimic joint=panda_finger_joint1 -> (none)

Commit message: update to 0.6.2

File: src/curobo/content/assets/robot/franka_description/franka_panda.urdf (robot description, URDF)
Before this commit: robot panda, 14 links, 13 joints
Joints:
- joint panda_finger_joint2: axis 0 1 0 -> 0 -1 0; limit lower=-0.04 upper=0.0 effort=20 velocity=0.2 -> lower=0.0 upper=0.04 effort=20 velocity=0.2

File: src/curobo/content/assets/robot/franka_description/franka_panda_mobile_xy_tz.urdf (robot description, URDF)
Before this commit: robot panda, 19 links, 18 joints
Joints:
- joint panda_finger_joint2: axis 0 1 0 -> 0 -1 0; limit lower=-0.04 upper=0.0 effort=20 velocity=0.2 -> lower=0.0 upper=0.04 effort=20 velocity=0.2; mimic (none) -> joint=panda_finger_joint1

Commit message: fix franka urdf issue

File: src/curobo/content/assets/robot/franka_description/franka_panda.urdf (robot description, URDF)
Before this commit: robot panda, 14 links, 13 joints
Joints:
- joint panda_finger_joint2: axis 0 -1 0 -> 0 1 0; origin xyz=0 0 0.0584 rpy=0 0 0 -> xyz=0 0 0.0584 rpy=0 0 3.14159265359
